File: Lily60.kicad_pcb (KiCad board)
At the start: 2 copper layers, 286.8 x 105 mm, 168 parts, among them J2 Conn_01x04, U1 RP2040, U2 XC6206PxxxMR, U3 W25Q128JVS, U4 SRV05-4, Y1 ABM8-272-T3

Commit message: V1.1
Parts:
- R4, R5, R6, R7: footprint hjcustom:C_0402_1005Metric_noref -> hjcustom:C_0402_1005Metric
Routing:
- net /QSPI_SS: track 21.2 -> 20.1 mm
- net /QSPI_SD2: track 14.8 -> 13.7 mm
- net /QSPI_SD1: track 15.9 -> 14.8 mm
- net GND: vias 95 -> 96
Other:
- board size 286.8 x 105 mm -> 286.8 x 104.2 mm
