File: Lily60.kicad_pcb (KiCad board)
At the start: 2 copper layers, 286.8 x 104.2 mm, 168 parts, among them J2 Conn_01x04, U1 RP2040, U2 XC6206PxxxMR, U3 W25Q128JVS, U4 SRV05-4, Y1 ABM8-272-T3

Commit message: change the PCB shape to non leaf version
Other:
- outline, holes or cut-outs redrawn
