File: Lily60.kicad_sch (KiCad schematic)
At the start: 162 parts, among them J2 Conn_01x04, U1 RP2040, U2 XC6206PxxxMR, U3 W25Q128JVS, U4 SRV05-4, Y1 ABM8-272-T3

Commit message: V1.1
Parts:
- R4, R5, R6, R7: footprint hjcustom:C_0402_1005Metric_noref -> hjcustom:C_0402_1005Metric
Changed lines of the file:
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@@
 			)
 		)
-		(property "Footprint" "hjcustom:C_0402_1005Metric_noref"
+		(property "Footprint" "hjcustom:C_0402_1005Metric"
 			(at 156.21 185.42 0)
 			(effects
@@
 			)
 		)
-		(property "Footprint" "hjcustom:C_0402_1005Metric_noref"
+		(property "Footprint" "hjcustom:C_0402_1005Metric"
 			(at 53.34 142.24 0)
 			(effects
@@
 			)
 		)
-		(property "Footprint" "hjcustom:C_0402_1005Metric_noref"
+		(property "Footprint" "hjcustom:C_0402_1005Metric"
 			(at 34.29 96.52 0)
 			(effects
@@
 			)
 		)
-		(property "Footprint" "hjcustom:C_0402_1005Metric_noref"
+		(property "Footprint" "hjcustom:C_0402_1005Metric"
 			(at 39.37 101.6 0)
 			(effects
